Commit message: change deprecated elements for noetic. added filem from arbotix repository

File: widowx_arm_description/robots/widowx_arm.urdf.xacro (robot description, xacro)
@@ -2,4 +2,10 @@
 <robot name="widowx_arm" xmlns:xacro="http://ros.org/wiki/xacro">
 	<xacro:include filename="$(find widowx_arm_description)/urdf/widowx.urdf.xacro"/>
+	 <link name="world" />
+	 <joint name="world_joint" type="fixed">
+		<parent link="world" />
+		<child link = "base_footprint" />
+		<origin xyz="0.0 0.0 0.0" rpy="0.0 0.0 0.0" />
+	 </joint>
 	<link name="base_footprint">
 		<visual>

Commit message: Upadate widowx_arm.urdf.xacro

File: widowx_arm_description/robots/widowx_arm.urdf.xacro (robot description, xacro)
@@ -1,11 +1,6 @@
 <?xml version="1.0" ?>
-<robot name="widowx_arm" xmlns:xacro="http://ros.org/wiki/xacro">
-	<xacro:include filename="$(find widowx_arm_description)/urdf/widowx.urdf.xacro"/>
-	 <link name="world" />
-	 <joint name="world_joint" type="fixed">
-		<parent link="world" />
-		<child link = "base_footprint" />
-		<origin xyz="0.0 0.0 0.0" rpy="0.0 0.0 0.0" />
-	 </joint>
+<robot xmlns:xacro="http://www.ros.org/wiki/xacro" name="widowx_arm">
+<xacro:include filename="$(find widowx_arm_description)/urdf/common_materials.xacro" />
+	<link name="world"/>
 	<link name="base_footprint">
 		<visual>
@@ -16,6 +11,13 @@
 		</visual>
 	</link>
-	<xacro:widowx_arm parent="base_footprint" prefix="">
-		<origin xyz="0.0 0.0 0.0" rpy="0.0 0.0 0.0"/>
-	</xacro:widowx_arm>
+	<joint name="fixed" type="fixed">
+    	<origin xyz="0 0 0" rpy="0 0 0"/>
+    	<parent link="world"/>
+    	<child link="base_footprint"/>
+  	</joint>
+	<xacro:include filename="$(find widowx_arm_description)/urdf/widowx.urdf.xacro"/>
+	<xacro:widowx_arm parent="base_footprint">
+    	<origin xyz="0 0 0" rpy="0 0 0" />
+    </xacro:widowx_arm>
+	<xacro:include filename="$(find widowx_arm_description)/urdf/gazebo_plugins.xacro"/>
 </robot>
