Commit message: Updated widowx.xacro
In this version the 'gripper_aux_link' is commented

File: widowx_arm_description/urdf/widowx.urdf.xacro (robot description, xacro)
@@ -4,12 +4,7 @@
    <xacro:property name="M_PI" value="3.14159"/>
    <xacro:include filename="$(find widowx_arm_description)/urdf/common_materials.xacro" />
-   <!--link name="plate_top_link"/-->
-   <!--joint name="fixed" type="fixed">
-      <parent link="plate_top_link" />
-      <child link="ph_base_link" />
-   </joint-->
-   <xacro:macro name="widowx_arm" params="parent prefix *origin">
+   <xacro:macro name="widowx_arm" params="parent *origin">
       <!-- links -->
-      <link name="${prefix}arm_base_link">
+      <link name="arm_base_link">
          <visual>
             <origin xyz="0 0 0" rpy="0 0 0" />
@@ -27,9 +22,9 @@
          <inertial>
             <origin xyz="0 0 0" rpy="0 0 0" />
-            <mass value="1" />
-            <inertia ixx="1.0" ixy="0.0" ixz="0.0" iyy="1.0" iyz="0.0" izz="1.0" />
-         </inertial>
-      </link>
-      <link name="${prefix}shoulder_link">
+            <mass value="0.01" />
+            <inertia ixx="1.0" ixy="0.0" ixz="0.0" iyy="1.0" iyz="0.0" izz="1.0" />
+         </inertial>
+      </link>
+      <link name="shoulder_link">
          <visual>
             <origin xyz="0 0 0" rpy="0 0 0" />
@@ -47,11 +42,11 @@
          <inertial>
             <origin xyz="0 0 0" rpy="0 0 0" />
-            <mass value="1" />
-            <inertia ixx="1.0" ixy="0.0" ixz="0.0" iyy="1.0" iyz="0.0" izz="1.0" />
-         </inertial>
-      </link>
-      <link name="${prefix}biceps_link">
-         <visual>
-			      <origin xyz="${M_SCALE*48.25} 0 ${M_SCALE*140}" rpy="0 0 0" />
+            <mass value="0.01" />
+            <inertia ixx="1.0" ixy="0.0" ixz="0.0" iyy="1.0" iyz="0.0" izz="1.0" />
+         </inertial>
+      </link>
+      <link name="biceps_link">
+         <visual>
+		<origin xyz="${M_SCALE*48.25} 0 ${M_SCALE*140}" rpy="0 0 0" />
             <!--origin xyz="0 0 0" rpy="0 0 0" /-->
             <geometry>
@@ -68,9 +63,9 @@
          <inertial>
             <origin xyz="0 0 0" rpy="0 0 0" />
-            <mass value="1" />
-            <inertia ixx="1.0" ixy="0.0" ixz="0.0" iyy="1.0" iyz="0.0" izz="1.0" />
-         </inertial>
-      </link>
-      <link name="${prefix}forearm_link">
+            <mass value="0.01" />
+            <inertia ixx="1.0" ixy="0.0" ixz="0.0" iyy="1.0" iyz="0.0" izz="1.0" />
+         </inertial>
+      </link>
+      <link name="forearm_link">
          <visual>
 			      <origin xyz="0 0 ${M_SCALE*142.03}" rpy="0 0 0" />
@@ -89,9 +84,9 @@
          <inertial>
             <origin xyz="0 0 0" rpy="0 0 0" />
-            <mass value="1" />
+            <mass value="0.01" />
             <inertia ixx="1.0" ixy="0.0" ixz="0.0" iyy="1.0" iyz="0.0" izz="1.0"/>
          </inertial>
       </link>
-      <link name="${prefix}wrist_1_link">
+      <link name="wrist_1_link">
          <visual>
             <origin xyz="0 0 0" rpy="0 0 0" />
@@ -109,9 +104,9 @@
          <inertial>
             <origin xyz="0 0 0" rpy="0 0 0" />
-            <mass value="1" />
-            <inertia ixx="1.0" ixy="0.0" ixz="0.0" iyy="1.0" iyz="0.0" izz="1.0" />
-         </inertial>
-      </link>
-      <link name="${prefix}wrist_2_link">
+            <mass value="0.01" />
+            <inertia ixx="1.0" ixy="0.0" ixz="0.0" iyy="1.0" iyz="0.0" izz="1.0" />
+         </inertial>
+      </link>
+      <link name="wrist_2_link">
          <visual>
             <origin xyz="0 0 ${M_SCALE*43}" rpy="0 0 0" />
@@ -129,9 +124,9 @@
          <inertial>
             <origin xyz="0 0 0" rpy="0 0 0" />
-            <mass value="1" />
-            <inertia ixx="1.0" ixy="0.0" ixz="0.0" iyy="1.0" iyz="0.0" izz="1.0" />
-         </inertial>
-      </link>
-      <link name="${prefix}gripper_rail_link">
+            <mass value="0.01" />
+            <inertia ixx="1.0" ixy="0.0" ixz="0.0" iyy="1.0" iyz="0.0" izz="1.0" />
+         </inertial>
+      </link>
+      <link name="gripper_rail_link">
          <visual>
             <origin xyz="0 0 0" rpy="0 0 1.57" />
@@ -149,11 +144,10 @@
          <inertial>
             <origin xyz="0 0 0" rpy="0 0 0" />
-            <mass value="1" />
-            <inertia ixx="1.0" ixy="0.0" ixz="0.0" iyy="1.0" iyz="0.0" izz="1.0" />
-         </inertial>
-      </link>
-      <link name="${prefix}gripper_aux_link">
-      </link>
-      <link name="${prefix}gripper_1_link">
+            <mass value="0.01" />
+            <inertia ixx="1.0" ixy="0.0" ixz="0.0" iyy="1.0" iyz="0.0" izz="1.0" />
+         </inertial>
+      </link>
+      <!--link name="gripper_aux_link"/-->
+      <link name="gripper_1_link">
          <visual>
             <origin xyz="0 -0.0007 0" rpy="0 0 1.57" />
@@ -171,9 +165,9 @@
          <inertial>
             <origin xyz="0 0 0" rpy="0 0 0" />
-            <mass value="1" />
-            <inertia ixx="1.0" ixy="0.0" ixz="0.0" iyy="1.0" iyz="0.0" izz="1.0" />
-         </inertial>
-      </link>
-      <link name="${prefix}gripper_2_link">
+            <mass value="0.01" />
+            <inertia ixx="1.0" ixy="0.0" ixz="0.0" iyy="1.0" iyz="0.0" izz="1.0" />
+         </inertial>
+      </link>
+      <link name="gripper_2_link">
          <visual>
             <origin xyz="0 0.0007 0" rpy="0 0 -1.57" />
@@ -191,127 +185,79 @@
          <inertial>
             <origin xyz="0 0 0" rpy="0 0 0" />
-            <mass value="1" />
+            <mass value="0.01" />
             <inertia ixx="1.0" ixy="0.0" ixz="0.0" iyy="1.0" iyz="0.0" izz="1.0" />
          </inertial>
       </link>
       <!-- joints -->
-      <joint name="${prefix}arm_base_joint" type="fixed">
+      <joint name="arm_base_joint" type="fixed">
          <insert_block name="origin" />
          <parent link="${parent}" />
-         <child link="${prefix}arm_base_link"/>
-      </joint>
-      <joint name="${prefix}joint_1" type="revolute">
+         <child link="arm_base_link"/>
+      </joint>
+      <joint name="joint_1" type="revolute">
          <origin xyz="0 0 ${M_SCALE*125}" rpy="0 0 0" />
-         <parent link="${prefix}arm_base_link" />
-         <child link="${prefix}shoulder_link" />
+         <parent link="arm_base_link" />
+         <child link="shoulder_link" />
          <axis xyz="0 0 1" />
          <limit lower="-2.617" upper="2.617" effort="0" velocity="0.785" />
       </joint>
-      <joint name="${prefix}joint_2" type="revolute">
+      <joint name="joint_2" type="revolute">
          <!--origin xyz="0.04825 0 0.14203" rpy="0 0 0" /-->
          <origin xyz="0 0 0" rpy="0 0 0" />
-         <parent link="${prefix}shoulder_link" />
-         <child link="${prefix}biceps_link" />
+         <parent link="shoulder_link" />
+         <child link="biceps_link" />
          <axis xyz="0 1 0" />
          <limit lower="-1.571" upper="1.571" effort="0" velocity="1.571" />
       </joint>
-      <joint name="${prefix}joint_3" type="revolute">
+      <joint name="joint_3" type="revolute">
          <origin xyz="${M_SCALE*48.25} 0 ${M_SCALE*142.03}" rpy="0 ${M_PI/2.0} 0" />
-         <parent link="${prefix}biceps_link" />
-         <child link="${prefix}forearm_link" />
+         <parent link="biceps_link" />
+         <child link="forearm_link" />
          <axis xyz="0 1 0" />
          <limit lower="-1.571" upper="1.571" effort="0" velocity="1.571" />
       </joint>
-      <joint name="${prefix}joint_4" type="revolute">
+      <joint name="joint_4" type="revolute">
          <origin xyz="0 0 ${M_SCALE*142.03}" rpy="0 0 0" />
-         <parent link="${prefix}forearm_link" />
-         <child link="${prefix}wrist_1_link" />
+         <parent link="forearm_link" />
+         <child link="wrist_1_link" />
          <axis xyz="0 1 0" />
          <limit lower="-1.745" upper="1.745" effort="0" velocity="1.571" />
       </joint>
-      <joint name="${prefix}joint_5" type="revolute">
+      <joint name="joint_5" type="revolute">
          <origin xyz="0 0 ${M_SCALE*71.5}" rpy="0 0 0" />
-         <parent link="${prefix}wrist_1_link" />
-         <child link="${prefix}wrist_2_link" />
+         <parent link="wrist_1_link" />
+         <child link="wrist_2_link" />
          <axis xyz="0 0 1" />
          <limit lower="-2.617" upper="2.617" effort="0" velocity="1.571" />
       </joint>
-      <joint name="${prefix}joint_6" type="fixed">
+      <joint name="joint_6" type="fixed">
          <origin xyz = "0 0 ${M_SCALE*43}" rpy="0 0 0" />
-         <parent link="${prefix}wrist_2_link" />
-         <child link="${prefix}gripper_rail_link" />
+         <parent link="wrist_2_link" />
+         <child link="gripper_rail_link" />
          <axis xyz="0 0 1" />
          <limit lower="-0.31" upper="0.1" effort="0" velocity="0.5" />
       </joint>
-      <joint name="${prefix}gripper_revolute_joint" type="revolute">
-         <origin xyz = "0 0 0" rpy="0 0 0" />
-         <parent link="${prefix}gripper_rail_link" />
-         <child link="${prefix}gripper_aux_link" />
-         <axis xyz="0 0 1" />
-         <limit lower="0" upper="2.6" effort="0" velocity="0.5" />
-      </joint>
-      <joint name="${prefix}gripper_prismatic_joint_1" type="prismatic">
+     <!--joint name="gripper_revolute_joint" type="revolute">
+         <origin rpy="0 0 0" xyz="0 0 0"/>
+         <parent link="gripper_rail_link"/>
+         <child link="gripper_aux_link"/>
+         <axis xyz="0 0 1"/>
+         <limit effort="0" lower="0" upper="2.6" velocity="0.5"/>
+      </joint-->
+      <joint name="gripper_prismatic_joint_1" type="prismatic">
          <origin xyz="0 0 0" rpy="0 0 0" />
-         <parent link="${prefix}gripper_rail_link" />
-         <child link="${prefix}gripper_1_link" />
+         <parent link="gripper_rail_link" />
+         <child link="gripper_1_link" />
          <axis xyz="0 -1 0" />
          <limit lower="0" upper="0.027" effort="0" velocity="0.5" />
       </joint>
-      <joint name="${prefix}gripper_prismatic_joint_2" type="prismatic">
+      <joint name="gripper_prismatic_joint_2" type="prismatic">
          <origin xyz="0 0 0" rpy="0 0 0" />
-         <parent link="${prefix}gripper_rail_link" />
-         <child link="${prefix}gripper_2_link" />
-         <mimic joint="${prefix}gripper_prismatic_joint_1" />
+         <parent link="gripper_rail_link" />
+         <child link="gripper_2_link" />
+         <mimic joint="gripper_prismatic_joint_1" />
          <axis xyz="0 1 0" />
          <limit lower="0" upper="0.027" effort="0" velocity="0.5" />
       </joint>
    </xacro:macro>
-  <transmission name="tran1">
-    <type>transmission_interface/SimpleTransmission</type>
-    <joint name="joint_1"/>
-    <actuator name="motor1">
-      <hardwareInterface>EffortJointInterface</hardwareInterface>
-      <mechanicalReduction>1</mechanicalReduction>
-    </actuator>
-  </transmission>
- <transmission name="tran2">
-    <type>transmission_interface/SimpleTransmission</type>
-    <joint name="joint_2"/>
-    <actuator name="motor2">
-      <hardwareInterface>EffortJointInterface</hardwareInterface>
-      <mechanicalReduction>1</mechanicalReduction>
-    </actuator>
-  </transmission>
- <transmission name="tran3">
-    <type>transmission_interface/SimpleTransmission</type>
-    <joint name="joint_3"/>
-    <actuator name="motor3">
-      <hardwareInterface>EffortJointInterface</hardwareInterface>
-      <mechanicalReduction>1</mechanicalReduction>
-    </actuator>
-  </transmission>
- <transmission name="tran4">
-    <type>transmission_interface/SimpleTransmission</type>
-    <joint name="joint_4"/>
-    <actuator name="motor4">
-      <hardwareInterface>EffortJointInterface</hardwareInterface>
-      <mechanicalReduction>1</mechanicalReduction>
-    </actuator>
-  </transmission>
- <transmission name="tran5">
-    <type>transmission_interface/SimpleTransmission</type>
-    <joint name="joint_6"/>
-    <actuator name="motor5">
-      <hardwareInterface>EffortJointInterface</hardwareInterface>
-      <mechanicalReduction>1</mechanicalReduction>
-    </actuator>
-  </transmission>
- <transmission name="tran6">
-    <type>transmission_interface/SimpleTransmission</type>
-    <joint name="gripper_prismatic_joint_1"/>
-    <actuator name="motor6">
-      <hardwareInterface>EffortJointInterface</hardwareInterface>
-      <mechanicalReduction>1</mechanicalReduction>
-    </actuator>
-  </transmission>
 </robot>

Commit message: Update widowx.urdf.xacro
Changed the "effort", set to 6

File: widowx_arm_description/urdf/widowx.urdf.xacro (robot description, xacro)
@@ -201,5 +201,5 @@
          <child link="shoulder_link" />
          <axis xyz="0 0 1" />
-         <limit lower="-2.617" upper="2.617" effort="0" velocity="0.785" />
+         <limit lower="-2.617" upper="2.617" effort="6" velocity="0.785" />
       </joint>
       <joint name="joint_2" type="revolute">
@@ -209,5 +209,5 @@
          <child link="biceps_link" />
          <axis xyz="0 1 0" />
-         <limit lower="-1.571" upper="1.571" effort="0" velocity="1.571" />
+         <limit lower="-1.571" upper="1.571" effort="6" velocity="1.571" />
       </joint>
       <joint name="joint_3" type="revolute">
@@ -216,5 +216,5 @@
          <child link="forearm_link" />
          <axis xyz="0 1 0" />
-         <limit lower="-1.571" upper="1.571" effort="0" velocity="1.571" />
+         <limit lower="-1.571" upper="1.571" effort="6" velocity="1.571" />
       </joint>
       <joint name="joint_4" type="revolute">
@@ -223,5 +223,5 @@
          <child link="wrist_1_link" />
          <axis xyz="0 1 0" />
-         <limit lower="-1.745" upper="1.745" effort="0" velocity="1.571" />
+         <limit lower="-1.745" upper="1.745" effort="6" velocity="1.571" />
       </joint>
       <joint name="joint_5" type="revolute">
@@ -230,5 +230,5 @@
          <child link="wrist_2_link" />
          <axis xyz="0 0 1" />
-         <limit lower="-2.617" upper="2.617" effort="0" velocity="1.571" />
+         <limit lower="-2.617" upper="2.617" effort="6" velocity="1.571" />
       </joint>
       <joint name="joint_6" type="fixed">
@@ -237,5 +237,5 @@
          <child link="gripper_rail_link" />
          <axis xyz="0 0 1" />
-         <limit lower="-0.31" upper="0.1" effort="0" velocity="0.5" />
+         <limit lower="-0.31" upper="0.1" effort="6" velocity="0.5" />
       </joint>
      <!--joint name="gripper_revolute_joint" type="revolute">
@@ -251,5 +251,5 @@
          <child link="gripper_1_link" />
          <axis xyz="0 -1 0" />
-         <limit lower="0" upper="0.027" effort="0" velocity="0.5" />
+         <limit lower="0" upper="0.027" effort="6" velocity="0.5" />
       </joint>
       <joint name="gripper_prismatic_joint_2" type="prismatic">
@@ -259,5 +259,5 @@
          <mimic joint="gripper_prismatic_joint_1" />
          <axis xyz="0 1 0" />
-         <limit lower="0" upper="0.027" effort="0" velocity="0.5" />
+         <limit lower="0" upper="0.027" effort="6" velocity="0.5" />
       </joint>
    </xacro:macro>
