Commit message: Fixing the shaking with the controllers
Adding the new .stl files of University of Cincinnati.

File: widowx_arm_description/urdf/widowx.urdf.xacro (robot description, xacro)
@@ -5,5 +5,4 @@
    <xacro:include filename="$(find widowx_arm_description)/urdf/common_materials.xacro" />
    <xacro:macro name="widowx_arm" params="parent *origin">
-      <xacro:include filename="$(find widowx_arm_description)/urdf/gazebo_plugins.xacro"/>
       <!-- links -->
       <link name="arm_base_link">
@@ -23,6 +22,6 @@
          <inertial>
             <origin xyz="0 0 0" rpy="0 0 0" />
-            <mass value="0.01" />
-            <inertia ixx="1.0" ixy="0.0" ixz="0.0" iyy="1.0" iyz="0.0" izz="1.0" />
+            <mass value="0.540142" />
+            <inertia ixx="0.0021190000" iyy="0.0006925000" izz="0.0025280000" ixy="-0.0000172100" ixz="0.0000006389" iyz="0.0000461200" />
          </inertial>
       </link>
@@ -42,36 +41,34 @@
          </collision>
          <inertial>
-            <origin xyz="0 0 0" rpy="0 0 0" />
-            <mass value="0.01" />
-            <inertia ixx="1.0" ixy="0.0" ixz="0.0" iyy="1.0" iyz="0.0" izz="1.0" />
+            <origin xyz="0.0 0.0 -0.04" rpy="0 0 0" />
+            <mass value="0.061" />
+            <inertia ixx="0.001" ixy="0.0" ixz="0.0" iyy="0.001" iyz="0.0" izz="0.001" />
          </inertial>
       </link>
       <link name="biceps_link">
          <visual>
-		<origin xyz="${M_SCALE*48.25} 0 ${M_SCALE*140}" rpy="0 0 0" />
-            <!--origin xyz="0 0 0" rpy="0 0 0" /-->
-            <geometry>
-               <mesh filename="package://widowx_arm_description/meshes/biceps_link.stl" />
-            </geometry>
-            <xacro:material_black />
-         </visual>
-         <collision>
-            <origin xyz="0 0 0" rpy="0 0 0" />
-            <geometry>
-               <mesh filename="package://widowx_arm_description/meshes/biceps_link.stl" />
-            </geometry>
-         </collision>
-         <inertial>
-            <origin xyz="0 0 0" rpy="0 0 0" />
-            <mass value="0.01" />
-            <inertia ixx="1.0" ixy="0.0" ixz="0.0" iyy="1.0" iyz="0.0" izz="1.0" />
+            <origin xyz="0 0 0" rpy="0 0 0" />
+            <geometry>
+               <mesh filename="package://widowx_arm_description/meshes/biceps_link.new.stl" />
+            </geometry>
+            <xacro:material_black />
+         </visual>
+         <collision>
+            <origin xyz="0 0 0" rpy="0 0 0" />
+            <geometry>
+               <mesh filename="package://widowx_arm_description/meshes/biceps_link.new.stl" />
+            </geometry>
+         </collision>
+         <inertial>
+            <origin xyz="0.006670 0.0 0.083394" rpy="0 0 0" />
+            <mass value="3.62e-1" />
+            <inertia ixx="0.001" ixy="0.0" ixz="0.0" iyy="0.001" iyz="0.0" izz="0.001" />
          </inertial>
       </link>
       <link name="forearm_link">
          <visual>
-			      <origin xyz="0 0 ${M_SCALE*142.03}" rpy="0 0 0" />
-			<!--origin xyz="0 0 0" rpy="0 0 0" /-->
-            <geometry>
-               <mesh filename="package://widowx_arm_description/meshes/forearm_link.stl"/>
+            <origin xyz="0 0 0" rpy="0 0 0" />
+            <geometry>
+               <mesh filename="package://widowx_arm_description/meshes/forearm_link.new.stl"/>
             </geometry>
            <xacro:material_black />
@@ -80,11 +77,11 @@
             <origin xyz="0 0 0" rpy="0 0 0" />
             <geometry>
-               <mesh filename="package://widowx_arm_description/meshes/forearm_link.stl"/>
-            </geometry>
-         </collision>
-         <inertial>
-            <origin xyz="0 0 0" rpy="0 0 0" />
-            <mass value="0.01" />
-            <inertia ixx="1.0" ixy="0.0" ixz="0.0" iyy="1.0" iyz="0.0" izz="1.0"/>
+               <mesh filename="package://widowx_arm_description/meshes/forearm_link.new.stl"/>
+            </geometry>
+         </collision>
+         <inertial>
+            <origin xyz="0.000018 0.0 0.090995" rpy="0 0 0" />
+            <mass value="1.87e-1" />
+            <inertia ixx="0.001" ixy="0.0" ixz="0.0" iyy="0.001" iyz="0.0" izz="0.001" />
          </inertial>
       </link>
@@ -104,29 +101,30 @@
          </collision>
          <inertial>
-            <origin xyz="0 0 0" rpy="0 0 0" />
-            <mass value="0.01" />
-            <inertia ixx="1.0" ixy="0.0" ixz="0.0" iyy="1.0" iyz="0.0" izz="1.0" />
+            <origin xyz="-0.010852 0.0 0.048078" rpy="0 0 0" />
+            <mass value="9.1e-2" />
+            <inertia ixx="0.001" ixy="0.0" ixz="0.0" iyy="0.001" iyz="0.0" izz="0.001" />
          </inertial>
       </link>
       <link name="wrist_2_link">
          <visual>
-            <origin xyz="0 0 ${M_SCALE*43}" rpy="0 0 0" />
-            <geometry>
-               <mesh filename="package://widowx_arm_description/meshes/wrist_2_link.stl"/>
-            </geometry>
-            <xacro:material_black />
-         </visual>
-         <collision>
-            <origin xyz="0 0 0" rpy="0 0 0" />
-            <geometry>
-               <mesh filename="package://widowx_arm_description/meshes/wrist_2_link.stl"/>
-            </geometry>
-         </collision>
-         <inertial>
-            <origin xyz="0 0 0" rpy="0 0 0" />
-            <mass value="0.01" />
-            <inertia ixx="1.0" ixy="0.0" ixz="0.0" iyy="1.0" iyz="0.0" izz="1.0" />
-         </inertial>
-      </link>
+            <origin xyz="0 0 0" rpy="0 0 0" />
+            <geometry>
+               <mesh filename="package://widowx_arm_description/meshes/wrist_2_link.new.stl"/>
+            </geometry>
+            <xacro:material_black />
+         </visual>
+         <collision>
+            <origin xyz="0 0 0" rpy="0 0 0" />
+            <geometry>
+               <mesh filename="package://widowx_arm_description/meshes/wrist_2_link.new.stl"/>
+            </geometry>
+         </collision>
+         <inertial>
+            <origin xyz="-0.018000 0.0 0.01500 " rpy="0 0 0" />
+            <mass value="6.3e-2" />
+            <inertia ixx="0.001" ixy="0.0" ixz="0.0" iyy="0.001" iyz="0.0" izz="0.001" />
+         </inertial>
+      </link>
+      <!-- gripper links -->
       <link name="gripper_rail_link">
          <visual>
@@ -137,17 +135,17 @@
             <xacro:material_black />
          </visual>
-         <collision>
-            <origin xyz="0 0 0" rpy="0 0 0" />
+         <!--Removed for now due to problems with collision in Gazebo-->
+         <!--collision>
+            <origin xyz="0 0 0" rpy="0 0 1.57" />
             <geometry>
                <mesh filename="package://widowx_arm_description/meshes/gripper_rail_link.stl"/>
             </geometry>
-         </collision>
-         <inertial>
-            <origin xyz="0 0 0" rpy="0 0 0" />
-            <mass value="0.01" />
-            <inertia ixx="1.0" ixy="0.0" ixz="0.0" iyy="1.0" iyz="0.0" izz="1.0" />
-         </inertial>
-      </link>
-      <!--link name="gripper_aux_link"/-->
+         </collision-->
+         <inertial>
+            <origin xyz="0 0 0" rpy="0 0 0" />
+            <mass value="7.0e-3" />
+            <inertia ixx="0.001" ixy="0.0" ixz="0.0" iyy="0.001" iyz="0.0" izz="0.001" />
+         </inertial>
+      </link>
       <link name="gripper_1_link">
          <visual>
@@ -159,13 +157,13 @@
          </visual>
          <collision>
-            <origin xyz="0 0 0" rpy="0 0 0" />
-            <geometry>
-               <mesh filename="package://widowx_arm_description/meshes/gripper_hand_fixed_link.stl"/>
-            </geometry>
-         </collision>
-         <inertial>
-            <origin xyz="0 0 0" rpy="0 0 0" />
-            <mass value="0.01" />
-            <inertia ixx="1.0" ixy="0.0" ixz="0.0" iyy="1.0" iyz="0.0" izz="1.0" />
+            <origin xyz="0 -0.0007 0" rpy="0 0 1.57" />
+            <geometry>
+               <mesh filename="package://widowx_arm_description/meshes/gripper_hand_fixed_link.stl"/>
+            </geometry>
+         </collision>
+         <inertial>
+            <origin xyz="0.0 -0.008292 0.017304" rpy="0 0 0" />
+            <mass value="8.0e-3" />
+            <inertia ixx="0.001" ixy="0.0" ixz="0.0" iyy="0.001" iyz="0.0" izz="0.001" />
          </inertial>
       </link>
@@ -179,13 +177,13 @@
          </visual>
          <collision>
-            <origin xyz="0 0 0" rpy="0 0 0" />
-            <geometry>
-               <mesh filename="package://widowx_arm_description/meshes/gripper_hand_fixed_link.stl"/>
-            </geometry>
-         </collision>
-         <inertial>
-            <origin xyz="0 0 0" rpy="0 0 0" />
-            <mass value="0.01" />
-            <inertia ixx="1.0" ixy="0.0" ixz="0.0" iyy="1.0" iyz="0.0" izz="1.0" />
+            <origin xyz="0 0.0007 0" rpy="0 0 -1.57" />
+            <geometry>
+               <mesh filename="package://widowx_arm_description/meshes/gripper_hand_fixed_link.stl"/>
+            </geometry>
+         </collision>
+         <inertial>
+            <origin xyz="0.0 0.008292 0.017304" rpy="0 0 0" />
+            <mass value="8.0e-3" />
+            <inertia ixx="0.001" ixy="0.0" ixz="0.0" iyy="0.001" iyz="0.0" izz="0.001" />
          </inertial>
       </link>
@@ -236,14 +234,5 @@
          <parent link="wrist_2_link" />
          <child link="gripper_rail_link" />
-         <axis xyz="0 0 1" />
-         <limit lower="-0.31" upper="0.1" effort="6" velocity="0.5" />
-      </joint>
-     <!--joint name="gripper_revolute_joint" type="revolute">
-         <origin rpy="0 0 0" xyz="0 0 0"/>
-         <parent link="gripper_rail_link"/>
-         <child link="gripper_aux_link"/>
-         <axis xyz="0 0 1"/>
-         <limit effort="0" lower="0" upper="2.6" velocity="0.5"/>
-      </joint-->
+      </joint>
       <joint name="gripper_prismatic_joint_1" type="prismatic">
          <origin xyz="0 0 0" rpy="0 0 0" />
@@ -251,5 +240,5 @@
          <child link="gripper_1_link" />
          <axis xyz="0 -1 0" />
-         <limit lower="0" upper="0.027" effort="6" velocity="0.5" />
+         <limit lower="0.002" upper="0.031" effort="6" velocity="0.5" />
       </joint>
       <joint name="gripper_prismatic_joint_2" type="prismatic">
@@ -259,5 +248,5 @@
          <mimic joint="gripper_prismatic_joint_1" />
          <axis xyz="0 1 0" />
-         <limit lower="0" upper="0.027" effort="6" velocity="0.5" />
+         <limit lower="0.002" upper="0.031" effort="6" velocity="0.5" />
       </joint>
    </xacro:macro>
